Commit message: Added lidar, simulation launch, and updated robot description

File: description/robot.urdf.xacro (robot description, xacro)
@@ -2,3 +2,4 @@
 <robot xmlns:xacro="http://www.ros.org/wiki/xacro"  name="robot">
   <xacro:include filename="$(find Ros_lidar_bot)/description/robot_core.xacro"/>
+  <xacro:include filename="$(find Ros_lidar_bot)/description/robot_control.xacro"/>
 </robot>

File: description/robot_core.xacro (robot description, xacro)
@@ -1,8 +1,7 @@
 <?xml version = "1.0"?>
 <robot xmlns:xacro="http://www.ros.org/wiki/xacro">
-<xacro:include filename="$(find Ros_lidar_bot)/description/inertial_macros.xacro"/>
 <xacro:include filename="inertial_macros.xacro"/>
 <!-- Base link -->
-<link name = "base_link">
+<link name="base_link">
 </link>
 <!--Chassis-->
@@ -33,65 +32,84 @@
 </link>
 <!-- Left wheel -->
-<joint name = "left_wheel_joint" type = "continuous">
-    <parent link = "base_link"/>
-    <child link = "left_wheel"/>
-    <origin xyz = "0 0.2 0" rpy = "0 0 0"/>
-    <axis xyz = "0 1 0"/>
+<joint name="left_wheel_joint" type="continuous">
+  <parent link="base_link"/>
+  <child link="left_wheel"/>
+  <!-- Wheel position relative to base -->
+  <origin xyz="0 0.175 0" rpy="0 0 0"/>
+  <!-- Wheel rotates about Y axis -->
+  <axis xyz="0 1 0"/>
 </joint>
-<link name = "left_wheel">
-    <visual>
-        <origin xyz = "0 0 0" rpy = "-1.5708 0 0"/>
-        <geometry>
-            <cylinder radius = "0.05" length = "0.05"/>
-        </geometry>
-        <material name = "red">
-            <color rgba = "1 0 0 1"/>
-        </material>
-    </visual>
-    <collision>
-        <origin xyz = "0 0 0" rpy = "-1.5708 0 0"/>
-        <geometry>
-            <cylinder radius = "0.05" length = "0.05"/>
-        </geometry>
-    </collision>
-    <xacro:inertial_cylinder mass = "0.1" length= "0.05" radius="0.05">
-        <origin xyz = "0 0 0" rpy = "-1.5708 0 0"/>
-    </xacro:inertial_cylinder>
+<link name="left_wheel">
+  <!-- VISUAL -->
+  <visual>
+    <!-- Rotate cylinder so it rolls on ground -->
+    <origin xyz = "0 0 0" rpy="-1.5708 0 0"/>
+    <geometry>
+      <cylinder radius="0.05" length="0.05"/>
+    </geometry>
+    <material name="red">
+      <color rgba="1 0 0 1"/>
+    </material>
+  </visual>
+  <!-- COLLISION -->
+  <collision>
+    <!-- MUST match visual orientation -->
+    <origin xyz ="0 0 0" rpy="-1.5708 0 0"/>
+    <geometry>
+      <cylinder radius="0.05" length="0.05"/>
+    </geometry>
+  </collision>
+  <!-- INERTIAL -->
+  <xacro:inertial_cylinder mass="0.1" length="0.05" radius="0.05">
+    <!-- MUST match visual/collision orientation -->
+    <origin xyz="0 0 0" rpy="-1.5708 0 0"/>
+  </xacro:inertial_cylinder>
 </link>
 <!-- right wheel -->
-<joint name = "right_wheel_joint" type = "continuous">
-    <parent link = "base_link"/>
-    <child link = "right_wheel"/>
-    <origin xyz = "0 -0.2 0" rpy = "0 0 0"/>
-    <axis xyz = "0 1 0"/>
+<!-- Right wheel -->
+<joint name="right_wheel_joint" type="continuous">
+  <parent link="base_link"/>
+  <child link="right_wheel"/>
+  <!-- Wheel position relative to base -->
+  <origin xyz="0 -0.175 0" rpy="0 0 0"/>
+  <!-- SAME axis as left wheel -->
+  <axis xyz="0 1 0"/>
 </joint>
-<link name = "right_wheel">
-    <visual>
-        <origin xyz = "0 0 0" rpy = "-1.5708 0 0"/>
-        <geometry>
-            <cylinder radius = "0.05" length = "0.05"/>
-        </geometry>
-        <material name = "red"/>
-    </visual>
-    <collision>
-        <origin xyz = "0 0 0" rpy = "-1.5708 0 0"/>
-        <geometry>
-            <cylinder radius = "0.05" length = "0.05"/>
-        </geometry>
-    </collision>
-    <xacro:inertial_cylinder mass = "0.1" length= "0.05" radius="0.05">
-        <origin xyz = "0 0 0" rpy = "-1.5708 0 0"/>
-    </xacro:inertial_cylinder>
+<link name="right_wheel">
+  <!-- VISUAL -->
+  <visual>
+    <!-- Rotate cylinder so it rolls on ground -->
+    <origin xyz="0 0 0" rpy="-1.5708 0 0"/>
+    <geometry>
+      <cylinder radius="0.05" length="0.05"/>
+    </geometry>
+    <material name="red">
+      <color rgba="1 0 0 1"/>
+    </material>
+  </visual>
+  <!-- COLLISION -->
+  <collision>
+    <!-- MUST match visual orientation -->
+    <origin xyz ="0 0 0" rpy="-1.5708 0 0"/>
+    <geometry>
+      <cylinder radius="0.05" length="0.05"/>
+    </geometry>
+  </collision>
+  <!-- INERTIAL -->
+  <xacro:inertial_cylinder mass="0.1" length="0.05" radius="0.05">
+    <!-- MUST match visual/collision orientation -->
+    <origin xyz="0 0 0" rpy="-1.5708 0 0"/>
+  </xacro:inertial_cylinder>
 </link>
 <joint name  = "lidar_joint" type = "fixed">
     <parent link = "chassis"/>
     <child link = "lidar_link"/>
-    <origin xyz = "0.1 0 0" rpy = "0 0 0"/>
+    <origin xyz = "0.2 0 0" rpy = "0 0 0"/>
 </joint>
 <link name = "lidar_link">
     <visual>
-        <origin xyz = "0.1 0 0.1"/>
+        <origin xyz = "0.2 0 0.1"/>
         <geometry>
-            <sphere radius = "0.02"/>
+            <cylinder radius = "0.07" length="0.09"/>
         </geometry>
         <material name = "green">
@@ -100,12 +118,12 @@
     </visual>
     <collision>
-        <origin xyz = "0.1 0 0.1"/>
+        <origin xyz = "0.2 0 0.1"/>
         <geometry>
-            <sphere radius = "0.02"/>
+            <cylinder radius = "0.07" length="0.09"/>
         </geometry>
     </collision>
-    <xacro:inertial_sphere mass = "0.01" radius="0.02">
-        <origin xyz ="0.1 0 0.1"/>
-    </xacro:inertial_sphere>
+    <xacro:inertial_cylinder mass = "0.01" length="0.09" radius="0.07">
+        <origin xyz ="0.2 0 0.1"/>
+    </xacro:inertial_cylinder>
 </link>
 <joint name  = "casterwheel" type = "fixed">
@@ -131,6 +149,42 @@
     </collision>
     <xacro:inertial_sphere mass = "0.04" radius="0.05">
-        <origin xyz ="0.3 0 0"/>
+        <origin xyz ="0.3 0 0" rpy="0 0 0"/>
     </xacro:inertial_sphere>
 </link>
+<gazebo>
+    <plugin
+      filename="libignition-gazebo-sensors-system.so"
+      name="gz::sim::systems::Sensors">
+      <render_engine>ogre2</render_engine>
+    </plugin>
+</gazebo>
+<gazebo reference="lidar_link">
+    <sensor name="gpu_lidar" type="gpu_lidar">
+      <pose>0 0 0 0 0 0</pose>
+      <topic>scan</topic>
+      <update_rate>8</update_rate>
+      <lidar>
+        <scan>
+          <horizontal>
+            <samples>720</samples>
+            <resolution>1</resolution>
+            <min_angle>-3.14</min_angle>
+            <max_angle>3.14</max_angle>
+          </horizontal>
+        </scan>
+        <range>
+          <min>0.01</min>
+          <max>12.0</max>
+          <resolution>0.005</resolution>
+        </range>
+        <noise>
+          <type>gaussian</type>
+          <mean>0.0</mean>
+          <stddev>0.001</stddev>
+        </noise>
+      </lidar>
+      <always_on>1</always_on>
+      <visualize>1</visualize>
+    </sensor>
+</gazebo>
 </robot>
