Commit message: lidar_completed

File: description/lidar.xacro (robot description, xacro)
@@ -1,31 +1,72 @@
-<?xml version = "1.0"?>
+<?xml version="1.0"?>
 <robot xmlns:xacro="http://www.ros.org/wiki/xacro">
+    <!-- LIDAR SENSOR -->
+    <!-- Lidar Joint -->
+    <joint name="laser_joint" type="fixed">
+        <parent link="chassis"/>
+        <child link="laser_frame"/>
+        <origin xyz="0.1 0 0.175" rpy="0 0 0"/>
+    </joint>
+    <!-- Lidar Link -->
+    <link name="laser_frame">
+        <visual>
+            <geometry>
+                <cylinder radius="0.05" length="0.04"/>
+            </geometry>
+            <material name="lidar_black">
+                <color rgba="0.1 0.1 0.1 1"/>
+            </material>
+        </visual>
+        <collision>
+            <geometry>
+                <cylinder radius="0.05" length="0.04"/>
+            </geometry>
+        </collision>
+        <inertial>
+            <origin xyz="0 0 0" rpy="0 0 0"/>
+            <mass value="0.1"/>
+            <inertia ixx="0.001" ixy="0" ixz="0" iyy="0.001" iyz="0" izz="0.001"/>
+        </inertial>
+    </link>
+    <!-- Gazebo Lidar Color -->
     <gazebo reference="laser_frame">
-        <material>Gazebo/Red</material>
-        <sensor name="laser" type="ray">
-            <pose> 0 0 0 0 0 0 </pose>
+        <material>Gazebo/Black</material>
+    </gazebo>
+    <!-- Ignition Gazebo Lidar Plugin (GPU Lidar sensor) -->
+    <gazebo reference="laser_frame">
+        <sensor name="gpu_lidar" type="gpu_lidar">
+            <pose>0 0 0 0 0 0</pose>
+            <topic>scan</topic>
+            <ignition_frame_id>laser_frame</ignition_frame_id>
+            <update_rate>10</update_rate>
             <visualize>true</visualize>
-            <update_rate>10</update_rate>
+            <always_on>true</always_on>
             <ray>
                 <scan>
                     <horizontal>
                         <samples>360</samples>
-                        <min_angle>-3.14</min_angle>
-                        <max_angle>3.14</max_angle>
+                        <resolution>1</resolution>
+                        <min_angle>-3.14159</min_angle>
+                        <max_angle>3.14159</max_angle>
                     </horizontal>
                 </scan>
                 <range>
                     <min>0.3</min>
-                    <max>12</max>
+                    <max>12.0</max>
+                    <resolution>0.01</resolution>
                 </range>
+                <noise>
+                    <type>gaussian</type>
+                    <mean>0.0</mean>
+                    <stddev>0.01</stddev>
+                </noise>
             </ray>
-            <plugin name="laser_controller" filename="libgazebo_ros_ray_sensor.so">
-                <ros>
-                    <argument>~/out:=scan</argument>
-                </ros>
-                <output_type>sensor_msgs/LaserScan</output_type>
-                <frame_name>laser_frame</frame_name>
-            </plugin>
         </sensor>
     </gazebo>
+    <!-- Ignition Gazebo Sensors Plugin (required to activate sensors) -->
+    <gazebo>
+        <plugin filename="libignition-gazebo-sensors-system.so" name="ignition::gazebo::systems::Sensors">
+            <render_engine>ogre2</render_engine>
+        </plugin>
+    </gazebo>
 </robot>

File: description/robot.urdf.xacro (robot description, xacro)
@@ -3,3 +3,4 @@
   <xacro:include filename="$(find Ros_lidar_bot)/description/robot_core.xacro"/>
   <xacro:include filename="$(find Ros_lidar_bot)/description/robot_control.xacro"/>
+  <xacro:include filename="$(find Ros_lidar_bot)/description/lidar.xacro"/>
 </robot>

File: description/robot_core.xacro (robot description, xacro)
@@ -102,29 +102,4 @@
   </xacro:inertial_cylinder>
 </link>
-<joint name  = "lidar_joint" type = "fixed">
-    <parent link = "chassis"/>
-    <child link = "lidar_link"/>
-    <origin xyz = "0.2 0 0" rpy = "0 0 0"/>
-</joint>
-<link name = "lidar_link">
-    <visual>
-        <origin xyz = "0.2 0 0.1"/>
-        <geometry>
-            <cylinder radius = "0.07" length="0.09"/>
-        </geometry>
-        <material name = "green">
-            <color rgba = "0 1 0 1"/>
-        </material>
-    </visual>
-    <collision>
-        <origin xyz = "0.2 0 0.1"/>
-        <geometry>
-            <cylinder radius = "0.07" length="0.09"/>
-        </geometry>
-    </collision>
-    <xacro:inertial_cylinder mass = "0.01" length="0.09" radius="0.07">
-        <origin xyz ="0.2 0 0.1"/>
-    </xacro:inertial_cylinder>
-</link>
 <joint name  = "casterwheel" type = "fixed">
     <parent link = "chassis"/>
@@ -152,39 +127,3 @@
     </xacro:inertial_sphere>
 </link>
-<gazebo>
-    <plugin
-      filename="libignition-gazebo-sensors-system.so"
-      name="gz::sim::systems::Sensors">
-      <render_engine>ogre2</render_engine>
-    </plugin>
-</gazebo>
-<gazebo reference="lidar_link">
-    <sensor name="gpu_lidar" type="gpu_lidar">
-      <pose>0 0 0 0 0 0</pose>
-      <topic>scan</topic>
-      <update_rate>8</update_rate>
-      <lidar>
-        <scan>
-          <horizontal>
-            <samples>720</samples>
-            <resolution>1</resolution>
-            <min_angle>-3.14</min_angle>
-            <max_angle>3.14</max_angle>
-          </horizontal>
-        </scan>
-        <range>
-          <min>0.01</min>
-          <max>12.0</max>
-          <resolution>0.005</resolution>
-        </range>
-        <noise>
-          <type>gaussian</type>
-          <mean>0.0</mean>
-          <stddev>0.001</stddev>
-        </noise>
-      </lidar>
-      <always_on>1</always_on>
-      <visualize>1</visualize>
-    </sensor>
-</gazebo>
 </robot>

Commit message: fixed wheel tfs

File: description/lidar.xacro (robot description, xacro)
@@ -6,5 +6,5 @@
         <parent link="chassis"/>
         <child link="laser_frame"/>
-        <origin xyz="0.1 0 0.175" rpy="0 0 0"/>
+        <origin xyz="0.1 0 0.15" rpy="0 0 0"/>
     </joint>
     <!-- Lidar Link -->

File: description/robot_control.xacro (robot description, xacro)
@@ -25,4 +25,9 @@
         <publish_wheel_tf>true</publish_wheel_tf>
   </plugin>
+  <plugin
+    filename="libgz-sim-joint-state-publisher-system.so"
+    name="gz::sim::systems::JointStatePublisher">
+    <topic>/joint_states</topic>
+  </plugin>
 </gazebo>
 <gazebo reference="caster_wheel">

Commit message: updated urdf

File: description/lidar.xacro (robot description, xacro)
@@ -3,29 +3,34 @@
     <!-- LIDAR SENSOR -->
     <!-- Lidar Joint -->
-    <joint name="laser_joint" type="fixed">
+    <!--joint name="laser_joint" type="fixed">
         <parent link="chassis"/>
         <child link="laser_frame"/>
         <origin xyz="0.1 0 0.15" rpy="0 0 0"/>
+    </joint-->
+    <joint name="laser_joint" type="fixed">
+        <origin xyz="-0.125 -0.073241 0.198241" rpy="0 0 0"/>
+        <parent link="base_link"/>
+        <child link="laser_frame"/>
     </joint>
     <!-- Lidar Link -->
     <link name="laser_frame">
+        <inertial>
+            <origin xyz="0.16 7.135009756631394e-08 0.01499992864990235" rpy="0 0 0"/>
+            <mass value="2.663442251713426"/>
+            <inertia ixx="0.002597" iyy="0.002597" izz="0.004794" ixy="0.0" iyz="0.0" ixz="0.0"/>
+        </inertial>
         <visual>
+            <origin xyz="0.125 0.073241 -0.198241" rpy="0 0 0"/>
             <geometry>
-                <cylinder radius="0.05" length="0.04"/>
+            <mesh filename="file://$(find Ros_lidar_bot)/meshes/lidar_1.stl" scale="0.001 0.001 0.001"/>
             </geometry>
-            <material name="lidar_black">
-                <color rgba="0.1 0.1 0.1 1"/>
-            </material>
+            <material name="silver"/>
         </visual>
         <collision>
+            <origin xyz="0.125 0.073241 -0.198241" rpy="0 0 0"/>
             <geometry>
-                <cylinder radius="0.05" length="0.04"/>
+            <mesh filename="file://$(find Ros_lidar_bot)/meshes/lidar_1.stl" scale="0.001 0.001 0.001"/>
             </geometry>
         </collision>
-        <inertial>
-            <origin xyz="0 0 0" rpy="0 0 0"/>
-            <mass value="0.1"/>
-            <inertia ixx="0.001" ixy="0" ixz="0" iyy="0.001" iyz="0" izz="0.001"/>
-        </inertial>
     </link>
     <!-- Gazebo Lidar Color -->

File: description/robot.urdf.xacro (robot description, xacro)
@@ -1,5 +1,5 @@
 <?xml version="1.0"?>
 <robot xmlns:xacro="http://www.ros.org/wiki/xacro"  name="robot">
-  <xacro:include filename="$(find Ros_lidar_bot)/description/robot_core.xacro"/>
+  <xacro:include filename="$(find Ros_lidar_bot)/description/slam.xacro"/>
   <xacro:include filename="$(find Ros_lidar_bot)/description/robot_control.xacro"/>
   <xacro:include filename="$(find Ros_lidar_bot)/description/lidar.xacro"/>

File: description/robot_control.xacro (robot description, xacro)
@@ -8,6 +8,6 @@
         <left_joint>left_wheel_joint</left_joint>
         <right_joint>right_wheel_joint</right_joint>
-        <wheel_separation>0.35</wheel_separation>
-        <wheel_radius>0.05</wheel_radius>
+        <wheel_separation>0.23</wheel_separation>
+        <wheel_radius>0.081</wheel_radius>
         <!-- limits -->
         <max_wheel_torque>200</max_wheel_torque>

Commit message: slam and our bot

File: description/lidar.xacro (robot description, xacro)
@@ -25,5 +25,7 @@
             <mesh filename="file://$(find Ros_lidar_bot)/meshes/lidar_1.stl" scale="0.001 0.001 0.001"/>
             </geometry>
-            <material name="silver"/>
+            <material name="silver">
+                <color rgba="0.00 0.00 0.00 1.0"/>   <!-- inline RGBA, no external file needed -->
+            </material>
         </visual>
         <collision>

File: description/slam.xacro (robot description, xacro)
@@ -14,5 +14,7 @@
       <mesh filename="file://$(find Ros_lidar_bot)/meshes/base_link.stl" scale="0.001 0.001 0.001"/>
     </geometry>
-    <material name="silver"/>
+    <material name="white">
+      <color rgba="1.0 1.0 1.0 1.0"/>
+    </material>
   </visual>
   <collision>
@@ -22,4 +24,11 @@
     </geometry>
   </collision>
+</link>
+<joint name = "base_footprint_joint" type= "fixed">
+    <parent link= "base_link"/>
+    <child link= "base_footprint"/>
+    <origin xyz = "0 0 0" rpy = "0 0 0"/>
+</joint>
+<link name = "base_footprint">
 </link>
 <link name="BHARAT_-FIH_-AMR-MAIN_WHEEL_WITH_MOTOR-PA-001__1__1">
@@ -34,5 +43,7 @@
       <mesh filename="file://$(find Ros_lidar_bot)/meshes/BHARAT_-FIH_-AMR-MAIN_WHEEL_WITH_MOTOR-PA-001__1__1.stl" scale="0.001 0.001 0.001"/>
     </geometry>
-    <material name="silver"/>
+    <material name="black">
+      <color rgba="0.00 0.00 0.00 1.0"/>
+    </material>
   </visual>
   <collision>
@@ -54,5 +65,7 @@
       <mesh filename="file://$(find Ros_lidar_bot)/meshes/BHARAT_-FIH_-AMR-MAIN_WHEEL_WITH_MOTOR-PA-001_1.stl" scale="0.001 0.001 0.001"/>
     </geometry>
-    <material name="silver"/>
+    <material name="black">
+      <color rgba="0.00 0.00 0.00 1.0"/>
+    </material>
   </visual>
   <collision>
@@ -74,5 +87,4 @@
       <mesh filename="file://$(find Ros_lidar_bot)/meshes/ball_caster_wheel__1__1.stl" scale="0.001 0.001 0.001"/>
     </geometry>
-    <material name="silver"/>
   </visual>
   <collision>
@@ -94,5 +106,4 @@
       <mesh filename="file://$(find Ros_lidar_bot)/meshes/ball_caster_wheel_1.stl" scale="0.001 0.001 0.001"/>
     </geometry>
-    <material name="silver"/>
   </visual>
   <collision>
