Commit message: IMU,Camera,Fixed Lidar, Map

File: description/lidar.xacro (robot description, xacro)
@@ -9,5 +9,5 @@
     </joint-->
     <joint name="laser_joint" type="fixed">
-        <origin xyz="-0.125 -0.073241 0.198241" rpy="0 0 0"/>
+        <origin xyz="-0.001839 0.002589 0.104922" rpy="0 0 0"/>
         <parent link="base_link"/>
         <child link="laser_frame"/>
@@ -16,28 +16,22 @@
     <link name="laser_frame">
         <inertial>
-            <origin xyz="0.16 7.135009756631394e-08 0.01499992864990235" rpy="0 0 0"/>
-            <mass value="2.663442251713426"/>
-            <inertia ixx="0.002597" iyy="0.002597" izz="0.004794" ixy="0.0" iyz="0.0" ixz="0.0"/>
+            <origin xyz="-4.0015749110241736e-07 -1.6278304991717424e-08 0.04331001637559857" rpy="0 0 0"/>
+    <mass value="0.5565046796809807"/>
+    <inertia ixx="0.000186" iyy="0.000186" izz="0.000341" ixy="0.0" iyz="0.0" ixz="-0.0"/>
         </inertial>
         <visual>
-            <origin xyz="0.125 0.073241 -0.198241" rpy="0 0 0"/>
+            <origin xyz="0.001839 -0.002589 -0.104922" rpy="0 0 0"/>
             <geometry>
-            <mesh filename="file://$(find Ros_lidar_bot)/meshes/lidar_1.stl" scale="0.001 0.001 0.001"/>
+            <mesh filename="file://$(find Ros_lidar_bot)/meshes/lidar_urdf_1.stl" scale="0.001 0.001 0.001"/>
             </geometry>
-            <material name="silver">
-                <color rgba="0.00 0.00 0.00 1.0"/>   <!-- inline RGBA, no external file needed -->
-            </material>
         </visual>
         <collision>
-            <origin xyz="0.125 0.073241 -0.198241" rpy="0 0 0"/>
+            <origin xyz="0.001839 -0.002589 -0.104922" rpy="0 0 0"/>
             <geometry>
-            <mesh filename="file://$(find Ros_lidar_bot)/meshes/lidar_1.stl" scale="0.001 0.001 0.001"/>
+            <mesh filename="file://$(find Ros_lidar_bot)/meshes/lidar_urdf_1.stl" scale="0.001 0.001 0.001"/>
             </geometry>
         </collision>
     </link>
     <!-- Gazebo Lidar Color -->
-    <gazebo reference="laser_frame">
-        <material>Gazebo/Black</material>
-    </gazebo>
     <!-- Ignition Gazebo Lidar Plugin (GPU Lidar sensor) -->
     <gazebo reference="laser_frame">
@@ -46,5 +40,5 @@
             <topic>scan</topic>
             <ignition_frame_id>laser_frame</ignition_frame_id>
-            <update_rate>10</update_rate>
+            <update_rate>20</update_rate>
             <visualize>true</visualize>
             <always_on>true</always_on>
@@ -72,8 +66,3 @@
     </gazebo>
     <!-- Ignition Gazebo Sensors Plugin (required to activate sensors) -->
-    <gazebo>
-        <plugin filename="libignition-gazebo-sensors-system.so" name="ignition::gazebo::systems::Sensors">
-            <render_engine>ogre2</render_engine>
-        </plugin>
-    </gazebo>
 </robot>

File: description/robot.urdf.xacro (robot description, xacro)
@@ -4,3 +4,5 @@
   <xacro:include filename="$(find Ros_lidar_bot)/description/robot_control.xacro"/>
   <xacro:include filename="$(find Ros_lidar_bot)/description/lidar.xacro"/>
+  <xacro:include filename="$(find Ros_lidar_bot)/description/camera.xacro"/>
+  <xacro:include filename="$(find Ros_lidar_bot)/description/imu.xacro"/>
 </robot>

File: description/robot_control.xacro (robot description, xacro)
@@ -8,5 +8,5 @@
         <left_joint>left_wheel_joint</left_joint>
         <right_joint>right_wheel_joint</right_joint>
-        <wheel_separation>0.23</wheel_separation>
+        <wheel_separation>0.3395</wheel_separation>
         <wheel_radius>0.081</wheel_radius>
         <!-- limits -->
@@ -14,13 +14,13 @@
         <max_wheel_acceleration>10.0</max_wheel_acceleration>
         <frame_id>odom</frame_id>
-        <child_frame_id>base_link</child_frame_id>
+        <child_frame_id>base_footprint</child_frame_id>
         <tf_topic>/tf</tf_topic>
         <odom_topic>/odom</odom_topic>
         <!-- outputs-->
-        <robot_base_frame>base_link</robot_base_frame>
+        <robot_base_frame>base_footprint</robot_base_frame>
         <!-- topics-->
         <topic>cmd_vel</topic>
         <publish_odom>true</publish_odom>
-        <publish_odom_tf>true</publish_odom_tf>
+        <publish_odom_tf>false</publish_odom_tf>
         <publish_wheel_tf>true</publish_wheel_tf>
   </plugin>
@@ -32,6 +32,6 @@
 </gazebo>
 <gazebo reference="caster_wheel">
-  <mu1 value="0.1"/>
-  <mu2 value="0.1"/>
+  <mu1 value="0.001"/>
+  <mu2 value="0.001"/>
 </gazebo>
 </robot>

File: description/slam.xacro (robot description, xacro)
@@ -1,11 +1,10 @@
 <?xml version="1.0" ?>
 <robot name="slam" xmlns:xacro="http://www.ros.org/wiki/xacro">
-<xacro:include filename="$(find Ros_lidar_bot)/description/materials.xacro" />
 <xacro:include filename="$(find Ros_lidar_bot)/description/slam.gazebo" />
 <link name="base_link">
   <inertial>
-    <origin xyz="-0.12499450936127811 -0.0732393668268621 0.25843254250315395" rpy="0 0 0"/>
-    <mass value="11.269909330356606"/>
-    <inertia ixx="0.1243" iyy="0.218253" izz="0.256396" ixy="-2e-06" iyz="-0.0" ixz="3e-06"/>
+    <origin xyz="-0.0019297244191736867 0.0018747496550703066 0.06995619724607677" rpy="0 0 0"/>
+    <mass value="21.04115508065235"/>
+    <inertia ixx="0.188108" iyy="0.289502" izz="0.293599" ixy="-0.000208" iyz="-0.000266" ixz="-7.4e-05"/>
   </inertial>
   <visual>
@@ -26,20 +25,20 @@
 </link>
 <joint name = "base_footprint_joint" type= "fixed">
-    <parent link= "base_link"/>
-    <child link= "base_footprint"/>
+    <parent link= "base_footprint"/>
+    <child link= "base_link"/>
     <origin xyz = "0 0 0" rpy = "0 0 0"/>
 </joint>
 <link name = "base_footprint">
 </link>
-<link name="BHARAT_-FIH_-AMR-MAIN_WHEEL_WITH_MOTOR-PA-001__1__1">
+<link name="wheel_urdf_1">
   <inertial>
-    <origin xyz="7.392549115040059e-06 -0.04111510772339333 -1.6452849457837537e-07" rpy="0 0 0"/>
-    <mass value="7.7692039603760845"/>
-    <inertia ixx="0.01318" iyy="0.022658" izz="0.013179" ixy="-3e-06" iyz="0.0" ixz="0.0"/>
+    <origin xyz="-4.001574910018034e-07 -0.05000001627830493 -4.836244008737944e-07" rpy="0 0 0"/>
+    <mass value="7.44298937241317"/>
+    <inertia ixx="0.013521" iyy="0.024417" izz="0.013521" ixy="-0.0" iyz="0.0" ixz="0.0"/>
   </inertial>
   <visual>
-    <origin xyz="0.125 0.188241 -0.226241" rpy="0 0 0"/>
+    <origin xyz="0.001839 0.112411 -0.034922" rpy="0 0 0"/>
     <geometry>
-      <mesh filename="file://$(find Ros_lidar_bot)/meshes/BHARAT_-FIH_-AMR-MAIN_WHEEL_WITH_MOTOR-PA-001__1__1.stl" scale="0.001 0.001 0.001"/>
+      <mesh filename="file://$(find Ros_lidar_bot)/meshes/wheel_urdf_1.stl" scale="0.001 0.001 0.001"/>
     </geometry>
     <material name="black">
@@ -48,20 +47,20 @@
   </visual>
   <collision>
-    <origin xyz="0.125 0.188241 -0.226241" rpy="0 0 0"/>
+    <origin xyz="0.001839 0.112411 -0.034922" rpy="0 0 0"/>
     <geometry>
-      <mesh filename="file://$(find Ros_lidar_bot)/meshes/BHARAT_-FIH_-AMR-MAIN_WHEEL_WITH_MOTOR-PA-001__1__1.stl" scale="0.001 0.001 0.001"/>
+      <mesh filename="file://$(find Ros_lidar_bot)/meshes/wheel_urdf_1.stl" scale="0.001 0.001 0.001"/>
     </geometry>
   </collision>
 </link>
-<link name="BHARAT_-FIH_-AMR-MAIN_WHEEL_WITH_MOTOR-PA-001_1">
+<link name="wheel_urdf__1__1">
   <inertial>
-    <origin xyz="-7.3925491141657584e-06 0.04011525042358858 -1.6452849452286422e-07" rpy="0 0 0"/>
-    <mass value="7.7692039603760845"/>
-    <inertia ixx="0.01318" iyy="0.022658" izz="0.013179" ixy="-3e-06" iyz="-0.0" ixz="-0.0"/>
+    <origin xyz="-4.0015749095214694e-07 0.04999998372169512 -4.836244007905277e-07" rpy="0 0 0"/>
+    <mass value="7.44298937241317"/>
+    <inertia ixx="0.013521" iyy="0.024417" izz="0.013521" ixy="0.0" iyz="0.0" ixz="-0.0"/>
   </inertial>
   <visual>
-    <origin xyz="0.125 -0.041759 -0.226241" rpy="0 0 0"/>
+    <origin xyz="0.001839 -0.117589 -0.034922" rpy="0 0 0"/>
     <geometry>
-      <mesh filename="file://$(find Ros_lidar_bot)/meshes/BHARAT_-FIH_-AMR-MAIN_WHEEL_WITH_MOTOR-PA-001_1.stl" scale="0.001 0.001 0.001"/>
+      <mesh filename="file://$(find Ros_lidar_bot)/meshes/wheel_urdf__1__1.stl" scale="0.001 0.001 0.001"/>
     </geometry>
     <material name="black">
@@ -70,7 +69,7 @@
   </visual>
   <collision>
-    <origin xyz="0.125 -0.041759 -0.226241" rpy="0 0 0"/>
+    <origin xyz="0.001839 -0.117589 -0.034922" rpy="0 0 0"/>
     <geometry>
-      <mesh filename="file://$(find Ros_lidar_bot)/meshes/BHARAT_-FIH_-AMR-MAIN_WHEEL_WITH_MOTOR-PA-001_1.stl" scale="0.001 0.001 0.001"/>
+      <mesh filename="file://$(find Ros_lidar_bot)/meshes/wheel_urdf__1__1.stl" scale="0.001 0.001 0.001"/>
     </geometry>
   </collision>
@@ -78,10 +77,10 @@
 <link name="ball_caster_wheel__1__1">
   <inertial>
-    <origin xyz="6.938893903907228e-18 7.135010103576089e-08 -0.012099122560755626" rpy="0 0 0"/>
-    <mass value="0.14791134084474702"/>
-    <inertia ixx="2.2e-05" iyy="2e-05" izz="2.4e-05" ixy="-0.0" iyz="-0.0" ixz="0.0"/>
+    <origin xyz="-4.001574910317274e-07 -1.6278612177851592e-08 -0.012099534835058778" rpy="0 0 0"/>
+    <mass value="0.1479113408447469"/>
+    <inertia ixx="2.2e-05" iyy="2e-05" izz="2.4e-05" ixy="0.0" iyz="0.0" ixz="-0.0"/>
   </inertial>
   <visual>
-    <origin xyz="-0.04 0.073241 -0.174741" rpy="0 0 0"/>
+    <origin xyz="0.166839 -0.002589 0.016578" rpy="0 0 0"/>
     <geometry>
       <mesh filename="file://$(find Ros_lidar_bot)/meshes/ball_caster_wheel__1__1.stl" scale="0.001 0.001 0.001"/>
@@ -89,5 +88,5 @@
   </visual>
   <collision>
-    <origin xyz="-0.04 0.073241 -0.174741" rpy="0 0 0"/>
+    <origin xyz="0.166839 -0.002589 0.016578" rpy="0 0 0"/>
     <geometry>
       <mesh filename="file://$(find Ros_lidar_bot)/meshes/ball_caster_wheel__1__1.stl" scale="0.001 0.001 0.001"/>
@@ -97,10 +96,10 @@
 <link name="ball_caster_wheel_1">
   <inertial>
-    <origin xyz="0.0 7.135010100800532e-08 -0.012099122560755599" rpy="0 0 0"/>
-    <mass value="0.14791134084474702"/>
-    <inertia ixx="2.2e-05" iyy="2e-05" izz="2.4e-05" ixy="0.0" iyz="-0.0" ixz="0.0"/>
+    <origin xyz="-4.001574910039718e-07 -1.627861223596483e-08 -0.012099534835058767" rpy="0 0 0"/>
+    <mass value="0.1479113408447469"/>
+    <inertia ixx="2.2e-05" iyy="2e-05" izz="2.4e-05" ixy="0.0" iyz="0.0" ixz="-0.0"/>
   </inertial>
   <visual>
-    <origin xyz="0.29 0.073241 -0.174741" rpy="0 0 0"/>
+    <origin xyz="-0.163161 -0.002589 0.016578" rpy="0 0 0"/>
     <geometry>
       <mesh filename="file://$(find Ros_lidar_bot)/meshes/ball_caster_wheel_1.stl" scale="0.001 0.001 0.001"/>
@@ -108,5 +107,5 @@
   </visual>
   <collision>
-    <origin xyz="0.29 0.073241 -0.174741" rpy="0 0 0"/>
+    <origin xyz="-0.163161 -0.002589 0.016578" rpy="0 0 0"/>
     <geometry>
       <mesh filename="file://$(find Ros_lidar_bot)/meshes/ball_caster_wheel_1.stl" scale="0.001 0.001 0.001"/>
@@ -114,23 +113,23 @@
   </collision>
 </link>
+<joint name="right_wheel_joint" type="continuous">
+  <origin xyz="-0.001839 -0.112411 0.034922" rpy="0 0 0"/>
+  <parent link="base_link"/>
+  <child link="wheel_urdf_1"/>
+  <axis xyz="0.0 1.0 0.0"/>
+</joint>
 <joint name="left_wheel_joint" type="continuous">
-  <origin xyz="-0.125 -0.188241 0.226241" rpy="0 0 0"/>
+  <origin xyz="-0.001839 0.117589 0.034922" rpy="0 0 0"/>
   <parent link="base_link"/>
-  <child link="BHARAT_-FIH_-AMR-MAIN_WHEEL_WITH_MOTOR-PA-001__1__1"/>
-  <axis xyz="0 1 0"/>
-</joint>
-<joint name="right_wheel_joint" type="continuous">
-  <origin xyz="-0.125 0.041759 0.226241" rpy="0 0 0"/>
-  <parent link="base_link"/>
-  <child link="BHARAT_-FIH_-AMR-MAIN_WHEEL_WITH_MOTOR-PA-001_1"/>
-  <axis xyz="0 1 0"/>
+  <child link="wheel_urdf__1__1"/>
+  <axis xyz="0.0 1.0 -0.0"/>
 </joint>
 <joint name="Rigid 3" type="fixed">
-  <origin xyz="0.04 -0.073241 0.174741" rpy="0 0 0"/>
+  <origin xyz="-0.166839 0.002589 -0.016578" rpy="0 0 0"/>
   <parent link="base_link"/>
   <child link="ball_caster_wheel__1__1"/>
 </joint>
 <joint name="Rigid 4" type="fixed">
-  <origin xyz="-0.29 -0.073241 0.174741" rpy="0 0 0"/>
+  <origin xyz="0.163161 0.002589 -0.016578" rpy="0 0 0"/>
   <parent link="base_link"/>
   <child link="ball_caster_wheel_1"/>
