Commit message: Changed world

File: description/camera.xacro (robot description, xacro)
@@ -4,5 +4,5 @@
     <parent link="base_link"/>
     <child link="camera_link"/>
-    <origin xyz="0.082 0 0.25" rpy="0 -0.5 0"/>
+    <origin xyz="0.082 0 0.25" rpy="0 0 0"/>
   </joint>
   <link name="camera_link">
